File: eagle/stm32l1.brd (EAGLE design)
At the start: 48 x 24.5 mm, 35 parts, among them IC1 STM32F405RGT, IC2 LT1763CS8-3.3, SW1 SWITCH_MCTAEF

Commit message: misc
Routing:
- net +5V: track 38.6 -> 35.0 mm
Other:
- board text added: "GD"
- board text added: "RX"
- board text added: "TX"
Changed lines of the file:
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@@
 <text x="33.8" y="25.3" size="0.7" layer="21" font="vector" ratio="13" rot="R90">SPI2_SCK</text>
 <text x="45.85" y="12" size="1.2" layer="22" font="vector" ratio="13" rot="MR0">STM32L1</text>
+<text x="3.75" y="5.5" size="0.7" layer="22" font="vector" ratio="13" rot="MR0">5V</text>
+<text x="3.75" y="8.1" size="0.7" layer="22" font="vector" ratio="13" rot="MR0">RX</text>
+<text x="3.65" y="10.6" size="0.7" layer="22" font="vector" ratio="13" rot="MR0">TX</text>
+<text x="3.55" y="13.2" size="0.7" layer="22" font="vector" ratio="13" rot="MR0">GD</text>
 </plain>
 <attributes>
@@
 <wire x1="2.1" y1="18.15" x2="2.125" y2="18.2" width="0.4064" layer="1"/>
 <wire x1="3.325" y1="18.15" x2="2.1" y2="18.15" width="0.4064" layer="1"/>
-<wire x1="2.075" y1="7.45" x2="2.075" y2="12.525" width="0.4064" layer="16"/>
-<wire x1="2.075" y1="12.525" x2="2.825" y2="13.275" width="0.4064" layer="16"/>
-<wire x1="2.825" y1="13.275" x2="4.2" y2="13.275" width="0.4064" layer="16"/>
-<wire x1="4.2" y1="13.275" x2="4.85" y2="13.925" width="0.4064" layer="16"/>
-<wire x1="4.0625" y1="5.4625" x2="2.075" y2="7.45" width="0.4064" layer="16"/>
 <via x="4.85" y="13.925" extent="1-16" drill="0.5"/>
-<wire x1="3.795" y1="5.73" x2="4.0625" y2="5.4625" width="0.4064" layer="1"/>
-<via x="4.0625" y="5.4625" extent="1-16" drill="0.6"/>
+<via x="5.4625" y="5.8625" extent="1-16" drill="0.6"/>
 <contactref element="U$1" pad="4"/>
 <contactref element="U$1" pad="4@1"/>
-<wire x1="1.0565" y1="5.89" x2="3.635" y2="5.89" width="0.4064" layer="1"/>
-<wire x1="3.635" y1="5.89" x2="4.0625" y2="5.4625" width="0.4064" layer="1"/>
-<wire x1="11.3435" y1="5.89" x2="4.49" y2="5.89" width="0.4064" layer="1"/>
-<wire x1="4.49" y1="5.89" x2="4.0625" y2="5.4625" width="0.4064" layer="1"/>
 <wire x1="13.24" y1="2.165" x2="13.24" y2="5.46" width="0.4064" layer="1"/>
 <wire x1="13.24" y1="5.46" x2="12.9" y2="5.8" width="0.4064" layer="1"/>
 <wire x1="12.9" y1="5.8" x2="12.81" y2="5.89" width="0.4064" layer="1"/>
 <wire x1="12.81" y1="5.89" x2="11.3435" y2="5.89" width="0.4064" layer="1"/>
+<wire x1="4.85" y1="13.925" x2="4.85" y2="6.475" width="0.4064" layer="16"/>
+<wire x1="4.85" y1="6.475" x2="5.4625" y2="5.8625" width="0.4064" layer="16"/>
+<wire x1="11.3435" y1="5.89" x2="5.49" y2="5.89" width="0.4064" layer="1"/>
+<wire x1="5.49" y1="5.89" x2="5.4625" y2="5.8625" width="0.4064" layer="1"/>
+<wire x1="1.0565" y1="5.89" x2="5.435" y2="5.89" width="0.4064" layer="1"/>
+<wire x1="5.435" y1="5.89" x2="5.4625" y2="5.8625" width="0.4064" layer="1"/>
 </signal>
 <signal name="N$18">

Commit message: misc
Routing:
- net BOOT: track 43.3 -> 33.3 mm
- net GND: track 36.5 -> 30.7 mm, vias 33 -> 34
Changed lines of the file:
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@@
 <layer number="21" name="tPlace" color="7" fill="1" visible="yes" active="yes"/>
 <layer number="22" name="bPlace" color="7" fill="1" visible="yes" active="yes"/>
-<layer number="23" name="tOrigins" color="15" fill="1" visible="no" active="yes"/>
-<layer number="24" name="bOrigins" color="15" fill="1" visible="no" active="yes"/>
+<layer number="23" name="tOrigins" color="15" fill="1" visible="yes" active="yes"/>
+<layer number="24" name="bOrigins" color="15" fill="1" visible="yes" active="yes"/>
 <layer number="25" name="tNames" color="10" fill="1" visible="yes" active="yes"/>
 <layer number="26" name="bNames" color="7" fill="1" visible="no" active="yes"/>
@@
 <text x="40.545" y="3.975" size="0.7" layer="25" font="vector" ratio="13">A6</text>
 <text x="43.22" y="3.975" size="0.7" layer="25" font="vector" ratio="13">A7</text>
-<text x="21.55" y="18.8" size="1.016" layer="22" font="vector" ratio="13" rot="MR0">seb@exse.net</text>
+<text x="18.35" y="9.9" size="1.016" layer="22" font="vector" ratio="13" rot="MR0">seb@exse.net</text>
 <text x="1.475" y="21.6" size="0.7" layer="25" font="vector" ratio="13" rot="SR90">GND</text>
 <text x="8.825" y="23.8" size="0.7" layer="25" font="vector" ratio="13" rot="SR180">3v3</text>
@@
 <text x="36.4" y="-11.8" size="0.7" layer="21" font="vector" ratio="13" rot="R90">UART3_RX</text>
 <text x="33.8" y="25.3" size="0.7" layer="21" font="vector" ratio="13" rot="R90">SPI2_SCK</text>
-<text x="45.85" y="12" size="1.2" layer="22" font="vector" ratio="13" rot="MR0">STM32L1</text>
+<text x="17.15" y="16.2" size="1.2" layer="22" font="vector" ratio="13" rot="MR0">STM32L1</text>
 <text x="3.75" y="5.5" size="0.7" layer="22" font="vector" ratio="13" rot="MR0">5V</text>
 <text x="3.75" y="8.1" size="0.7" layer="22" font="vector" ratio="13" rot="MR0">RX</text>
@@
 <wire x1="28.5" y1="8.7885" x2="28.5" y2="10.6" width="0.254" layer="1"/>
 <wire x1="28.5" y1="10.6" x2="27.62" y2="11.48" width="0.254" layer="1"/>
-<wire x1="27.62" y1="11.48" x2="27.62" y2="11.45" width="0.254" layer="1"/>
 <wire x1="29.1" y1="7.47" x2="29.82" y2="6.85" width="0.254" layer="16"/>
-<wire x1="29.1" y1="10.3" x2="29.1" y2="7.47" width="0.254" layer="16"/>
-<wire x1="28.35" y1="11.05" x2="29.1" y2="10.3" width="0.254" layer="16"/>
-<wire x1="27.62" y1="11.45" x2="28.35" y2="11.05" width="0.254" layer="16"/>
 <wire x1="27.62" y1="12.05" x2="26.195" y2="14.075" width="0.254" layer="16"/>
-<wire x1="27.62" y1="11.45" x2="27.62" y2="12.05" width="0.254" layer="16"/>
 <wire x1="26.195" y1="14.075" x2="26.095" y2="15.438" width="0.254" layer="1"/>
 <wire x1="26.775" y1="13.575" x2="28" y2="14.8" width="0.254" layer="1"/>
@@
 <wire x1="28.8" y1="19.8486" x2="29.642878125" y2="20.69141875" width="0.254" layer="1"/>
 <wire x1="28.8" y1="19.8" x2="28.8" y2="19.8486" width="0.254" layer="1"/>
-<wire x1="27.62" y1="11.45" x2="28.05" y2="11.45" width="0.254" layer="16"/>
 <wire x1="29.4" y1="19.2" x2="28.8" y2="19.8" width="0.254" layer="1"/>
 <wire x1="29.4" y1="18.6" x2="29.4" y2="19.2" width="0.254" layer="1"/>
@@
 <via x="45.17" y="5.725" extent="1-16" drill="0.5"/>
 <via x="44.37" y="17.85" extent="1-16" drill="0.5"/>
-<via x="27.62" y="11.45" extent="1-16" drill="0.5"/>
+<via x="25.82" y="11.45" extent="1-16" drill="0.5"/>
 <via x="26.195" y="14.075" extent="1-16" drill="0.5"/>
 <via x="42.27" y="18.425" extent="1-16" drill="0.5"/>
@@
 <via x="7.8" y="16.225" extent="1-16" drill="0.5"/>
 <via x="7.8" y="19.6" extent="1-16" drill="0.5"/>
-<via x="14.925" y="17.5" extent="1-16" drill="0.5"/>
+<via x="15.125" y="20.1" extent="1-16" drill="0.5"/>
 <via x="17.225" y="9.125" extent="1-16" drill="0.5"/>
-<via x="15.35" y="15.425" extent="1-16" drill="0.5"/>
-<via x="16.525" y="16.75" extent="1-16" drill="0.5"/>
+<via x="19.05" y="17.925" extent="1-16" drill="0.5"/>
+<via x="15.825" y="14.95" extent="1-16" drill="0.5"/>
 <via x="13.675" y="23.475" extent="1-16" drill="0.5"/>
 <via x="8.3" y="12.725" extent="1-16" drill="0.5"/>
@@
 <wire x1="30.706240625" y1="18.0657375" x2="31.365503125" y2="18.725" width="0.254" layer="1"/>
 <via x="30.625" y="17.425" extent="1-16" drill="0.5"/>
-<via x="30.125" y="14.525" extent="1-16" drill="0.5"/>
+<via x="31.425" y="14.525" extent="1-16" drill="0.5"/>
 <contactref element="U$1" pad="1"/>
 <contactref element="U$1" pad="1@1"/>
 <via x="20.095" y="11.675" extent="1-16" drill="0.5"/>
 <via x="14.395" y="5.175" extent="1-16" drill="0.5"/>
+<via x="29.025" y="14.725" extent="1-16" drill="0.5"/>
 <wire x1="31.506240625" y1="18.8657375" x2="31.365503125" y2="18.725" width="0" layer="19" extent="1-1"/>
 </signal>
@@
 <wire x1="43.1" y1="9.2" x2="45.325" y2="7.075" width="0.254" layer="1"/>
 <wire x1="43.1" y1="9.8" x2="43.1" y2="9.2" width="0.254" layer="1"/>
-<wire x1="23.6833" y1="12.9" x2="22.66740625" y2="13.9159875" width="0.254" layer="1"/>
-<wire x1="24.4" y1="12.9" x2="23.6833" y2="12.9" width="0.254" layer="1"/>
-<wire x1="24.8" y1="12.5" x2="24.4" y2="12.9" width="0.254" layer="1"/>
+<wire x1="23.5833" y1="13" x2="22.66740625" y2="13.9159875" width="0.254" layer="1"/>
+<wire x1="24.3" y1="13" x2="23.5833" y2="13" width="0.254" layer="1"/>
+<wire x1="24.8" y1="12.5" x2="24.3" y2="13" width="0.254" layer="1"/>
 <wire x1="29.8" y1="12.5" x2="24.8" y2="12.5" width="0.254" layer="1"/>
 <wire x1="18.965" y1="12.9291" x2="18.965" y2="12.835" width="0.6096" layer="16"/>
@@
 <wire x1="44.7" y1="9.8" x2="43.1" y2="9.8" width="0.254" layer="1"/>
 <wire x1="29.5" y1="17.5666" x2="29.5" y2="17.2" width="0.254" layer="1"/>
-<wire x1="29.5" y1="17.2" x2="28.9" y2="16.6" width="0.254" layer="1"/>
-<wire x1="28.9" y1="16.6" x2="28.9" y2="13.4" width="0.254" layer="1"/>
-<wire x1="28.9" y1="13.4" x2="29.8" y2="12.5" width="0.254" layer="1"/>
 <via x="15.2" y="11.9" extent="1-16" drill="0.6"/>
 <wire x1="14.5" y1="10" x2="14.5" y2="11.2" width="0.6096" layer="1"/>
@@
 <wire x1="13.5" y1="10.7" x2="15.2" y2="10.7" width="0.6096" layer="16"/>
 <wire x1="15.2" y1="10.7" x2="15.2" y2="11.9" width="0.6096" layer="16"/>
+<wire x1="29.8" y1="16.4" x2="29.7" y2="16.5" width="0.254" layer="1"/>
+<wire x1="29.7" y1="16.5" x2="29.5" y2="16.7" width="0.254" layer="1"/>
+<wire x1="29.5" y1="16.7" x2="29.5" y2="17.2" width="0.254" layer="1"/>
+<wire x1="29.8" y1="12.5" x2="30.1" y2="12.8" width="0.254" layer="1"/>
+<wire x1="30.1" y1="12.8" x2="30.1" y2="14.6" width="0.254" layer="1"/>
+<wire x1="30.1" y1="14.6" x2="30.1" y2="16.1" width="0.254" layer="1"/>
+<wire x1="30.1" y1="16.1" x2="29.5" y2="16.7" width="0.254" layer="1"/>
 </signal>
 <signal name="+5V">
@@
 <wire x1="25" y1="14.4118" x2="24.081621875" y2="15.330203125" width="0.254" layer="1"/>
 <wire x1="25" y1="14.3" x2="25" y2="14.4118" width="0.254" layer="1"/>
-<wire x1="25" y1="12.4" x2="25" y2="14.3" width="0.254" layer="16"/>
-<wire x1="27" y1="10.4" x2="25" y2="12.4" width="0.254" layer="16"/>
-<wire x1="27.9" y1="10.4" x2="27" y2="10.4" width="0.254" layer="16"/>
-<wire x1="28.5" y1="9.8" x2="27.9" y2="10.4" width="0.254" layer="16"/>
-<wire x1="28.5" y1="6.7" x2="28.5" y2="9.8" width="0.254" layer="16"/>
-<wire x1="29.6" y1="5.6" x2="28.5" y2="6.7" width="0.254" layer="16"/>
-<wire x1="29.6" y1="5.6" x2="30.7" y2="5.6" width="0.254" layer="16"/>
-<wire x1="30.7" y1="5.6" x2="31.3" y2="6.2" width="0.254" layer="16"/>
-<wire x1="31.3" y1="6.2" x2="31.3" y2="6.6" width="0.254" layer="16"/>
-<wire x1="31.3" y1="6.6" x2="29.8" y2="8.1" width="0.254" layer="16"/>
-<wire x1="29.8" y1="8.1" x2="29.8" y2="9.3" width="0.254" layer="16"/>
-<wire x1="29.8" y1="9.3" x2="32.2" y2="11.7" width="0.254" layer="16"/>
+<wire x1="25" y1="12.9" x2="25" y2="14.3" width="0.254" layer="16"/>
 <wire x1="32.2" y1="11.7" x2="34.8" y2="11.7" width="0.254" layer="16"/>
 <wire x1="34.8" y1="11.7" x2="38.3" y2="8.2" width="0.254" layer="16"/>
@@
 <wire x1="20" y1="20.3" x2="18.31" y2="21.99" width="0.254" layer="1"/>
 <wire x1="18.31" y1="21.99" x2="18.31" y2="22.485" width="0.254" layer="1"/>
+<wire x1="25" y1="12.9" x2="25.4" y2="12.5" width="0.254" layer="16"/>
+<wire x1="25.4" y1="12.5" x2="26.5" y2="12.5" width="0.254" layer="16"/>
+<wire x1="26.5" y1="12.5" x2="27.9" y2="11.1" width="0.254" layer="16"/>
+<wire x1="27.9" y1="11.1" x2="28.4" y2="11.1" width="0.254" layer="16"/>
+<wire x1="28.4" y1="11.1" x2="29.1" y2="10.4" width="0.254" layer="16"/>
+<wire x1="29.1" y1="10.4" x2="30.9" y2="10.4" width="0.254" layer="16"/>
+<wire x1="30.9" y1="10.4" x2="32.2" y2="11.7" width="0.254" layer="16"/>
 </signal>
 <signal name="B14">
@@
 <wire x1="26.1" y1="10.2" x2="25.95" y2="10.35" width="0.254" layer="1"/>
 <wire x1="25.95" y1="10.35" x2="25.35" y2="10.35" width="0.254" layer="1"/>
-<wire x1="25.35" y1="10.35" x2="24.4" y2="11.3" width="0.254" layer="1"/>
-<wire x1="24.4" y1="11.3" x2="23.9" y2="11.3" width="0.254" layer="1"/>
-<wire x1="23.9" y1="11.3" x2="23.4" y2="11.8" width="0.254" layer="1"/>
-<wire x1="23.4" y1="11.8" x2="21.5" y2="11.8" width="0.254" layer="1"/>
+<wire x1="25.35" y1="10.35" x2="24.6" y2="11.1" width="0.254" layer="1"/>
+<wire x1="24.6" y1="11.1" x2="24" y2="11.1" width="0.254" layer="1"/>
+<wire x1="24" y1="11.1" x2="23.3" y2="11.8" width="0.254" layer="1"/>
+<wire x1="23.3" y1="11.8" x2="21.5" y2="11.8" width="0.254" layer="1"/>
 <via x="26.1" y="10.2" extent="1-16" drill="0.4"/>
 <contactref element="C12" pad="1"/>
